File: RFID v0.1.sch (EAGLE design)
At the start: 32 parts, among them K1 G5LE, Q1 XTAL 16MHz, T1 BC817-40, U1 ARDUINOSPI-REFRENCE, U2 POWER-POD 5V0, U3 ATMEGA328P-MU, U4 POWER-POD 3V3

Commit message: Add early box design and some WIP board layout
Parts:
- added L1: (no value), CISECO eaglecad designs:INDUCTOR0603K-SMALL
Connections:
- new net VCC: C1.2, C6.2, L1.2, R3.2, U3.AVCC, U3.VCC@1, U3.VCC@2
- net 3V3: now also L1.1; no longer C1.2, C6.2, R3.2, U3.AVCC, U3.VCC@1, U3.VCC@2
